File: SHIELD_MEGA/gps_module.sch (KiCad schematic (older format))
At the start: 0 parts

Commit message: GPS connection
Parts:
- added J?: Conn_01x06_Female, symbol Connector:Conn_01x06_Female
Connections:
- new net 5V: J?.6 (Pin_6)
- new net GND: J?.1 (Pin_1)
- no-connect marks 0 -> 2
Changed lines of the file:
@@
 $Descr A4 11693 8268
 encoding utf-8
-Sheet 1 6
+Sheet 6 6
 Title ""
 Date ""
@@
 Comment4 ""
 $EndDescr
+NoConn ~ 5500 3400
+NoConn ~ 5500 3500
+Text Label 5200 3300 0    50   ~ 0
+GND
+Wire Wire Line
+	5200 3300 5500 3300
+$Comp
+L Connector:Conn_01x06_Female J?
+U 1 1 61960166
+P 5700 3500
+F 0 "J?" H 5728 3476 50  0000 L CNN
+F 1 "Conn_01x06_Female" H 5728 3385 50  0000 L CNN
+F 2 "" H 5700 3500 50  0001 C CNN
+F 3 "~" H 5700 3500 50  0001 C CNN
+	1    5700 3500
+	1    0    0    -1
+$EndComp
+Text Label 5200 3800 0    50   ~ 0
+5V
+Wire Wire Line
+	5200 3800 5500 3800
 $EndSCHEMATC
