File: SHIELD_MEGA/Radio_receiver.sch (KiCad schematic (older format))
At the start: 0 parts

Commit message: pins of radio receiver
Parts:
- added J? (x6): Conn_01x03_Female, symbol Connector:Conn_01x03_Female
Connections:
- new net 5V: J?.2 (Pin_2), J?.2 (Pin_2), J?.2 (Pin_2), J?.2 (Pin_2), J?.2 (Pin_2), J?.2 (Pin_2)
- new net D10: J?.1 (Pin_1)
- new net D11: J?.1 (Pin_1)
- new net D50: J?.1 (Pin_1)
- new net D51: J?.1 (Pin_1)
- new net D52: J?.1 (Pin_1)
- new net D53: J?.1 (Pin_1)
- new net GND: J?.3 (Pin_3), J?.3 (Pin_3), J?.3 (Pin_3), J?.3 (Pin_3), J?.3 (Pin_3), J?.3 (Pin_3)
Changed lines of the file:
@@
 Comment4 ""
 $EndDescr
+$Comp
+L Connector:Conn_01x03_Female J?
+U 1 1 61973E8C
+P 5750 3050
+F 0 "J?" H 5778 3076 50  0000 L CNN
+F 1 "Conn_01x03_Female" H 5778 2985 50  0000 L CNN
+F 2 "" H 5750 3050 50  0001 C CNN
+F 3 "~" H 5750 3050 50  0001 C CNN
+	1    5750 3050
+	1    0    0    -1
+$EndComp
+$Comp
+L Connector:Conn_01x03_Female J?
+U 1 1 61974EE4
+P 5750 3400
+F 0 "J?" H 5778 3426 50  0000 L CNN
+F 1 "Conn_01x03_Female" H 5778 3335 50  0000 L CNN
+F 2 "" H 5750 3400 50  0001 C CNN
+F 3 "~" H 5750 3400 50  0001 C CNN
+	1    5750 3400
+	1    0    0    -1
+$EndComp
+$Comp
+L Connector:Conn_01x03_Female J?
+U 1 1 6197586F
+P 5750 3750
+F 0 "J?" H 5778 3776 50  0000 L CNN
+F 1 "Conn_01x03_Female" H 5778 3685 50  0000 L CNN
+F 2 "" H 5750 3750 50  0001 C CNN
+F 3 "~" H 5750 3750 50  0001 C CNN
+	1    5750 3750
+	1    0    0    -1
+$EndComp
+$Comp
+L Connector:Conn_01x03_Female J?
+U 1 1 61975F3B
+P 5750 4150
+F 0 "J?" H 5778 4176 50  0000 L CNN
+F 1 "Conn_01x03_Female" H 5778 4085 50  0000 L CNN
+F 2 "" H 5750 4150 50  0001 C CNN
+F 3 "~" H 5750 4150 50  0001 C CNN
+	1    5750 4150
+	1    0    0    -1
+$EndComp
+$Comp
+L Connector:Conn_01x03_Female J?
+U 1 1 61976273
+P 5750 4550
+F 0 "J?" H 5778 4576 50  0000 L CNN
+F 1 "Conn_01x03_Female" H 5778 4485 50  0000 L CNN
+F 2 "" H 5750 4550 50  0001 C CNN
+F 3 "~" H 5750 4550 50  0001 C CNN
+	1    5750 4550
+	1    0    0    -1
+$EndComp
+$Comp
+L Connector:Conn_01x03_Female J?
+U 1 1 61976608
+P 5750 4950
+F 0 "J?" H 5778 4976 50  0000 L CNN
+F 1 "Conn_01x03_Female" H 5778 4885 50  0000 L CNN
+F 2 "" H 5750 4950 50  0001 C CNN
+F 3 "~" H 5750 4950 50  0001 C CNN
+	1    5750 4950
+	1    0    0    -1
+$EndComp
+Text Label 5300 5050 0    50   ~ 0
+GND
+Wire Wire Line
+	5300 5050 5550 5050
+Text Label 5300 4950 0    50   ~ 0
+5V
+Wire Wire Line
+	5300 4950 5550 4950
+Text Label 5300 4850 0    50   ~ 0
+D11
+Wire Wire Line
+	5300 4850 5550 4850
+Text Label 5300 4650 0    50   ~ 0
+GND
+Wire Wire Line
+	5300 4650 5550 4650
+Wire Wire Line
+	5550 4550 5300 4550
+Text Label 5300 4550 0    50   ~ 0
+5V
+Text Label 5300 4450 0    50   ~ 0
+D10
+Wire Wire Line
+	5300 4450 5550 4450
+Wire Wire Line
+	5550 4250 5300 4250
+Text Label 5300 4250 0    50   ~ 0
+GND
+Text Label 5300 4150 0    50   ~ 0
+5V
+Wire Wire Line
+	5300 4150 5550 4150
+Wire Wire Line
+	5550 4050 5300 4050
+Text Label 5300 4050 0    50   ~ 0
+D50
+Text Label 5300 3850 0    50   ~ 0
+GND
+Wire Wire Line
+	5300 3850 5550 3850
+Wire Wire Line
+	5550 3750 5300 3750
+Text Label 5300 3750 0    50   ~ 0
+5V
+Text Label 5300 3650 0    50   ~ 0
+D51
+Wire Wire Line
+	5300 3650 5550 3650
+Wire Wire Line
+	5550 3500 5300 3500
+Text Label 5300 3500 0    50   ~ 0
+GND
+Text Label 5300 3400 0    50   ~ 0
+5V
+Wire Wire Line
+	5300 3400 5550 3400
+Wire Wire Line
+	5550 3300 5300 3300
+Text Label 5300 3300 0    50   ~ 0
+D52
+Wire Wire Line
+	5550 3150 5300 3150
+Text Label 5300 3150 0    50   ~ 0
+GND
+Wire Wire Line
+	5300 3050 5550 3050
+Text Label 5300 3050 0    50   ~ 0
+5V
+Wire Wire Line
+	5300 2950 5550 2950
+Text Label 5300 2950 0    50   ~ 0
+D53
 $EndSCHEMATC
