File: SHIELD_MEGA/COMUNICATION_BUS.sch (KiCad schematic (older format))
At the start: 4 parts

Commit message: Defining ref number to parts in comunication sheet
Parts:
- gave numbers to parts that had none: 4
Changed lines of the file:
@@
 encoding utf-8
 Sheet 6 10
-Title ""
-Date ""
-Rev ""
-Comp ""
+Title "SHIELD ARDUINO MEGA"
+Date "2021-11-21"
+Rev "V1"
+Comp "PROEX - UNIFEI"
 Comment1 ""
 Comment2 ""
 Comment3 ""
-Comment4 ""
+Comment4 "LINCOLN WALLACE VELOSO ALMEIDA"
 $EndDescr
 Wire Wire Line
@@
 	5950 4950 5750 4950
 $Comp
-L Connector:Conn_01x04_Male J?
+L Connector:Conn_01x04_Male J9
 U 1 1 61C34CF1
 P 3550 3650
-F 0 "J?" H 3658 3931 50  0000 C CNN
+F 0 "J9" H 3658 3931 50  0000 C CNN
 F 1 "Conn_01x04_Male" H 3658 3840 50  0000 C CNN
 F 2 "" H 3550 3650 50  0001 C CNN
@@
 $EndComp
 $Comp
-L Connector:Conn_01x04_Male J?
+L Connector:Conn_01x04_Male J10
 U 1 1 61C36CF7
 P 5550 3650
-F 0 "J?" H 5658 3931 50  0000 C CNN
+F 0 "J10" H 5658 3931 50  0000 C CNN
 F 1 "Conn_01x04_Male" H 5658 3840 50  0000 C CNN
 F 2 "" H 5550 3650 50  0001 C CNN
@@
 $EndComp
 $Comp
-L Connector:Conn_01x04_Male J?
+L Connector:Conn_01x04_Male J12
 U 1 1 61C37472
 P 7500 3650
-F 0 "J?" H 7608 3931 50  0000 C CNN
+F 0 "J12" H 7608 3931 50  0000 C CNN
 F 1 "Conn_01x04_Male" H 7608 3840 50  0000 C CNN
 F 2 "" H 7500 3650 50  0001 C CNN
@@
 $EndComp
 $Comp
-L Connector:Conn_01x06_Male J?
+L Connector:Conn_01x06_Male J11
 U 1 1 61C38C33
 P 5550 5150
-F 0 "J?" H 5658 5531 50  0000 C CNN
+F 0 "J11" H 5658 5531 50  0000 C CNN
 F 1 "Conn_01x06_Male" H 5658 5440 50  0000 C CNN
 F 2 "" H 5550 5150 50  0001 C CNN
