File: SHIELD_MEGA/ACCEL.sch (KiCad schematic (older format))
At the start: 1 part

Commit message: Changing to female connector
Parts:
- removed J?: Conn_01x07_Male, symbol Connector:Conn_01x07_Male
- added J?: Conn_01x07_Female, symbol Connector:Conn_01x07_Female
Changed lines of the file:
@@
 $Descr A4 11693 8268
 encoding utf-8
-Sheet 2 9
+Sheet 2 10
 Title ""
 Date ""
@@
 Wire Wire Line
 	5800 3300 5650 3300
-$Comp
-L Connector:Conn_01x07_Male J?
-U 1 1 61961FB2
-P 5450 3300
-F 0 "J?" H 5550 3750 50  0000 C CNN
-F 1 "Conn_01x07_Male" V 5400 3300 50  0000 C CNN
-F 2 "" H 5450 3300 50  0001 C CNN
-F 3 "~" H 5450 3300 50  0001 C CNN
-	1    5450 3300
-	1    0    0    -1
-$EndComp
 Wire Wire Line
 	5650 3400 5800 3400
@@
 Text HLabel 5800 3400 2    50   Input ~ 0
 SDA
+$Comp
+L Connector:Conn_01x07_Female J?
+U 1 1 61B8ACF7
+P 5450 3300
+F 0 "J?" H 5342 2775 50  0000 C CNN
+F 1 "Conn_01x07_Female" H 5342 2866 50  0000 C CNN
+F 2 "" H 5450 3300 50  0001 C CNN
+F 3 "~" H 5450 3300 50  0001 C CNN
+	1    5450 3300
+	-1   0    0    1
+$EndComp
 $EndSCHEMATC

Commit message: Anotations in ACCEL sheet
Parts:
- gave numbers to parts that had none: 1
Changed lines of the file:
@@
 encoding utf-8
 Sheet 2 10
-Title ""
-Date ""
-Rev ""
-Comp ""
+Title "SHIELD ARDUINO MEGA"
+Date "2021-11-21"
+Rev "V1"
+Comp "PROEX - UNIFEI"
 Comment1 ""
 Comment2 ""
 Comment3 ""
-Comment4 ""
+Comment4 "LINCOLN WALLACE VELOSO ALMEIDA"
 $EndDescr
 NoConn ~ 5650 3000
@@
 SDA
 $Comp
-L Connector:Conn_01x07_Female J?
+L Connector:Conn_01x07_Female J3
 U 1 1 61B8ACF7
 P 5450 3300
-F 0 "J?" H 5342 2775 50  0000 C CNN
+F 0 "J3" H 5342 2775 50  0000 C CNN
 F 1 "Conn_01x07_Female" H 5342 2866 50  0000 C CNN
 F 2 "" H 5450 3300 50  0001 C CNN
