File: SHIELD_MEGA/ANALOG_BUS.sch (KiCad schematic (older format))
At the start: 16 parts, among them J13 Conn_01x03_Male, J14 Conn_01x03_Male, J15 Conn_01x03_Male, J16 Conn_01x03_Male, J17 Conn_01x03_Male, J18 Conn_01x03_Male, J19 Conn_01x03_Male, J20 Conn_01x03_Male, J21 Conn_01x03_Male, J22 Conn_01x03_Male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

Commit message: Updating ref's
Parts:
- J16: renamed from J13; footprint (none) -> Connector_PinHeader_2.54mm:PinHeader_1x03_P2.54mm_Vertical
- J17: renamed from J14; footprint (none) -> Connector_PinHeader_2.54mm:PinHeader_1x03_P2.54mm_Vertical
- J18: renamed from J15; footprint (none) -> Connector_PinHeader_2.54mm:PinHeader_1x03_P2.54mm_Vertical
- J19: renamed from J16; footprint (none) -> Connector_PinHeader_2.54mm:PinHeader_1x03_P2.54mm_Vertical
- J20: renamed from J17; footprint (none) -> Connector_PinHeader_2.54mm:PinHeader_1x03_P2.54mm_Vertical
- J21: renamed from J18; footprint (none) -> Connector_PinHeader_2.54mm:PinHeader_1x03_P2.54mm_Vertical
- J22: renamed from J19; footprint (none) -> Connector_PinHeader_2.54mm:PinHeader_1x03_P2.54mm_Vertical
- J23: renamed from J20; footprint (none) -> Connector_PinHeader_2.54mm:PinHeader_1x03_P2.54mm_Vertical
- J24: renamed from J21; footprint (none) -> Connector_PinHeader_2.54mm:PinHeader_1x03_P2.54mm_Vertical
- J25: renamed from J22; footprint (none) -> Connector_PinHeader_2.54mm:PinHeader_1x03_P2.54mm_Vertical
- J26: renamed from J23; footprint (none) -> Connector_PinHeader_2.54mm:PinHeader_1x03_P2.54mm_Vertical
- J27: renamed from J24; footprint (none) -> Connector_PinHeader_2.54mm:PinHeader_1x03_P2.54mm_Vertical
- J28: renamed from J25; footprint (none) -> Connector_PinHeader_2.54mm:PinHeader_1x03_P2.54mm_Vertical
- J29: renamed from J26; footprint (none) -> Connector_PinHeader_2.54mm:PinHeader_1x03_P2.54mm_Vertical
- J30: renamed from J27; footprint (none) -> Connector_PinHeader_2.54mm:PinHeader_1x03_P2.54mm_Vertical
- J31: renamed from J28; footprint (none) -> Connector_PinHeader_2.54mm:PinHeader_1x03_P2.54mm_Vertical
Changed lines of the file:
@@
 P 3100 2600
 AR Path="/6194FDB3/61A3708D" Ref="J?"  Part="1"
-AR Path="/6194FDB3/61A24149/61A3708D" Ref="J13"  Part="1"
-F 0 "J13" H 3200 2300 50  0000 C CNN
+AR Path="/6194FDB3/61A24149/61A3708D" Ref="J16"  Part="1"
+F 0 "J16" H 3200 2300 50  0000 C CNN
 F 1 "Conn_01x03_Male" H 3200 2400 50  0000 C CNN
-F 2 "" H 3100 2600 50  0001 C CNN
+F 2 "Connector_PinHeader_2.54mm:PinHeader_1x03_P2.54mm_Vertical" H 3100 2600 50  0001 C CNN
 F 3 "~" H 3100 2600 50  0001 C CNN
 	1    3100 2600
@@
 P 3100 3250
 AR Path="/6194FDB3/61A37097" Ref="J?"  Part="1"
-AR Path="/6194FDB3/61A24149/61A37097" Ref="J14"  Part="1"
-F 0 "J14" H 3250 2950 50  0000 C CNN
+AR Path="/6194FDB3/61A24149/61A37097" Ref="J17"  Part="1"
+F 0 "J17" H 3250 2950 50  0000 C CNN
 F 1 "Conn_01x03_Male" H 3250 3050 50  0000 C CNN
-F 2 "" H 3100 3250 50  0001 C CNN
+F 2 "Connector_PinHeader_2.54mm:PinHeader_1x03_P2.54mm_Vertical" H 3100 3250 50  0001 C CNN
 F 3 "~" H 3100 3250 50  0001 C CNN
 	1    3100 3250
@@
 P 3100 4600
 AR Path="/6194FDB3/61A370A1" Ref="J?"  Part="1"
-AR Path="/6194FDB3/61A24149/61A370A1" Ref="J16"  Part="1"
-F 0 "J16" H 3200 4300 50  0000 C CNN
+AR Path="/6194FDB3/61A24149/61A370A1" Ref="J19"  Part="1"
+F 0 "J19" H 3200 4300 50  0000 C CNN
 F 1 "Conn_01x03_Male" H 3250 4400 50  0000 C CNN
-F 2 "" H 3100 4600 50  0001 C CNN
+F 2 "Connector_PinHeader_2.54mm:PinHeader_1x03_P2.54mm_Vertical" H 3100 4600 50  0001 C CNN
 F 3 "~" H 3100 4600 50  0001 C CNN
 	1    3100 4600
@@
 P 3100 3950
 AR Path="/6194FDB3/61A370AB" Ref="J?"  Part="1"
-AR Path="/6194FDB3/61A24149/61A370AB" Ref="J15"  Part="1"
-F 0 "J15" H 3250 3650 50  0000 C CNN
+AR Path="/6194FDB3/61A24149/61A370AB" Ref="J18"  Part="1"
+F 0 "J18" H 3250 3650 50  0000 C CNN
 F 1 "Conn_01x03_Male" H 3250 3750 50  0000 C CNN
-F 2 "" H 3100 3950 50  0001 C CNN
+F 2 "Connector_PinHeader_2.54mm:PinHeader_1x03_P2.54mm_Vertical" H 3100 3950 50  0001 C CNN
 F 3 "~" H 3100 3950 50  0001 C CNN
 	1    3100 3950
@@
 P 4600 2600
 AR Path="/6194FDB3/61A370B5" Ref="J?"  Part="1"
-AR Path="/6194FDB3/61A24149/61A370B5" Ref="J17"  Part="1"
-F 0 "J17" H 4700 2300 50  0000 C CNN
+AR Path="/6194FDB3/61A24149/61A370B5" Ref="J20"  Part="1"
+F 0 "J20" H 4700 2300 50  0000 C CNN
 F 1 "Conn_01x03_Male" H 4700 2400 50  0000 C CNN
-F 2 "" H 4600 2600 50  0001 C CNN
+F 2 "Connector_PinHeader_2.54mm:PinHeader_1x03_P2.54mm_Vertical" H 4600 2600 50  0001 C CNN
 F 3 "~" H 4600 2600 50  0001 C CNN
 	1    4600 2600
@@
 P 4600 3250
 AR Path="/6194FDB3/61A370BF" Ref="J?"  Part="1"
-AR Path="/6194FDB3/61A24149/61A370BF" Ref="J18"  Part="1"
-F 0 "J18" H 4700 2950 50  0000 C CNN
+AR Path="/6194FDB3/61A24149/61A370BF" Ref="J21"  Part="1"
+F 0 "J21" H 4700 2950 50  0000 C CNN
 F 1 "Conn_01x03_Male" H 4700 3050 50  0000 C CNN
-F 2 "" H 4600 3250 50  0001 C CNN
+F 2 "Connector_PinHeader_2.54mm:PinHeader_1x03_P2.54mm_Vertical" H 4600 3250 50  0001 C CNN
 F 3 "~" H 4600 3250 50  0001 C CNN
 	1    4600 3250
@@
 P 4600 4600
 AR Path="/6194FDB3/61A370C9" Ref="J?"  Part="1"
-AR Path="/6194FDB3/61A24149/61A370C9" Ref="J20"  Part="1"
-F 0 "J20" H 4700 4300 50  0000 C CNN
+AR Path="/6194FDB3/61A24149/61A370C9" Ref="J23"  Part="1"
+F 0 "J23" H 4700 4300 50  0000 C CNN
 F 1 "Conn_01x03_Male" H 4700 4400 50  0000 C CNN
-F 2 "" H 4600 4600 50  0001 C CNN
+F 2 "Connector_PinHeader_2.54mm:PinHeader_1x03_P2.54mm_Vertical" H 4600 4600 50  0001 C CNN
 F 3 "~" H 4600 4600 50  0001 C CNN
 	1    4600 4600
@@
 P 4600 3950
 AR Path="/6194FDB3/61A370D3" Ref="J?"  Part="1"
-AR Path="/6194FDB3/61A24149/61A370D3" Ref="J19"  Part="1"
-F 0 "J19" H 4700 3650 50  0000 C CNN
+AR Path="/6194FDB3/61A24149/61A370D3" Ref="J22"  Part="1"
+F 0 "J22" H 4700 3650 50  0000 C CNN
 F 1 "Conn_01x03_Male" H 4700 3750 50  0000 C CNN
-F 2 "" H 4600 3950 50  0001 C CNN
+F 2 "Connector_PinHeader_2.54mm:PinHeader_1x03_P2.54mm_Vertical" H 4600 3950 50  0001 C CNN
 F 3 "~" H 4600 3950 50  0001 C CNN
 	1    4600 3950
@@
 P 6100 2600
 AR Path="/6194FDB3/61A370DD" Ref="J?"  Part="1"
-AR Path="/6194FDB3/61A24149/61A370DD" Ref="J21"  Part="1"
-F 0 "J21" H 6200 2300 50  0000 C CNN
+AR Path="/6194FDB3/61A24149/61A370DD" Ref="J24"  Part="1"
+F 0 "J24" H 6200 2300 50  0000 C CNN
 F 1 "Conn_01x03_Male" H 6200 2400 50  0000 C CNN
-F 2 "" H 6100 2600 50  0001 C CNN
+F 2 "Connector_PinHeader_2.54mm:PinHeader_1x03_P2.54mm_Vertical" H 6100 2600 50  0001 C CNN
 F 3 "~" H 6100 2600 50  0001 C CNN
 	1    6100 2600
@@
 P 6100 3250
 AR Path="/6194FDB3/61A370E7" Ref="J?"  Part="1"
-AR Path="/6194FDB3/61A24149/61A370E7" Ref="J22"  Part="1"
-F 0 "J22" H 6200 2950 50  0000 C CNN
+AR Path="/6194FDB3/61A24149/61A370E7" Ref="J25"  Part="1"
+F 0 "J25" H 6200 2950 50  0000 C CNN
 F 1 "Conn_01x03_Male" H 6200 3050 50  0000 C CNN
-F 2 "" H 6100 3250 50  0001 C CNN
+F 2 "Connector_PinHeader_2.54mm:PinHeader_1x03_P2.54mm_Vertical" H 6100 3250 50  0001 C CNN
 F 3 "~" H 6100 3250 50  0001 C CNN
 	1    6100 3250
@@
 P 6100 4600
 AR Path="/6194FDB3/61A370F1" Ref="J?"  Part="1"
-AR Path="/6194FDB3/61A24149/61A370F1" Ref="J24"  Part="1"
-F 0 "J24" H 6200 4300 50  0000 C CNN
+AR Path="/6194FDB3/61A24149/61A370F1" Ref="J27"  Part="1"
+F 0 "J27" H 6200 4300 50  0000 C CNN
 F 1 "Conn_01x03_Male" H 6200 4400 50  0000 C CNN
-F 2 "" H 6100 4600 50  0001 C CNN
+F 2 "Connector_PinHeader_2.54mm:PinHeader_1x03_P2.54mm_Vertical" H 6100 4600 50  0001 C CNN
 F 3 "~" H 6100 4600 50  0001 C CNN
 	1    6100 4600
@@
 P 6100 3950
 AR Path="/6194FDB3/61A370FB" Ref="J?"  Part="1"
-AR Path="/6194FDB3/61A24149/61A370FB" Ref="J23"  Part="1"
-F 0 "J23" H 6200 3650 50  0000 C CNN
+AR Path="/6194FDB3/61A24149/61A370FB" Ref="J26"  Part="1"
+F 0 "J26" H 6200 3650 50  0000 C CNN
 F 1 "Conn_01x03_Male" H 6200 3750 50  0000 C CNN
-F 2 "" H 6100 3950 50  0001 C CNN
+F 2 "Connector_PinHeader_2.54mm:PinHeader_1x03_P2.54mm_Vertical" H 6100 3950 50  0001 C CNN
 F 3 "~" H 6100 3950 50  0001 C CNN
 	1    6100 3950
@@
 P 7600 2600
 AR Path="/6194FDB3/61A37105" Ref="J?"  Part="1"
-AR Path="/6194FDB3/61A24149/61A37105" Ref="J25"  Part="1"
-F 0 "J25" H 7700 2300 50  0000 C CNN
+AR Path="/6194FDB3/61A24149/61A37105" Ref="J28"  Part="1"
+F 0 "J28" H 7700 2300 50  0000 C CNN
 F 1 "Conn_01x03_Male" H 7700 2400 50  0000 C CNN
-F 2 "" H 7600 2600 50  0001 C CNN
+F 2 "Connector_PinHeader_2.54mm:PinHeader_1x03_P2.54mm_Vertical" H 7600 2600 50  0001 C CNN
 F 3 "~" H 7600 2600 50  0001 C CNN
 	1    7600 2600
@@
 P 7600 3250
 AR Path="/6194FDB3/61A3710F" Ref="J?"  Part="1"
-AR Path="/6194FDB3/61A24149/61A3710F" Ref="J26"  Part="1"
-F 0 "J26" H 7700 2950 50  0000 C CNN
+AR Path="/6194FDB3/61A24149/61A3710F" Ref="J29"  Part="1"
+F 0 "J29" H 7700 2950 50  0000 C CNN
 F 1 "Conn_01x03_Male" H 7700 3050 50  0000 C CNN
-F 2 "" H 7600 3250 50  0001 C CNN
+F 2 "Connector_PinHeader_2.54mm:PinHeader_1x03_P2.54mm_Vertical" H 7600 3250 50  0001 C CNN
 F 3 "~" H 7600 3250 50  0001 C CNN
 	1    7600 3250
@@
 P 7600 4600
 AR Path="/6194FDB3/61A37119" Ref="J?"  Part="1"
-AR Path="/6194FDB3/61A24149/61A37119" Ref="J28"  Part="1"
-F 0 "J28" H 7700 4300 50  0000 C CNN
+AR Path="/6194FDB3/61A24149/61A37119" Ref="J31"  Part="1"
+F 0 "J31" H 7700 4300 50  0000 C CNN
 F 1 "Conn_01x03_Male" H 7700 4400 50  0000 C CNN
-F 2 "" H 7600 4600 50  0001 C CNN
+F 2 "Connector_PinHeader_2.54mm:PinHeader_1x03_P2.54mm_Vertical" H 7600 4600 50  0001 C CNN
 F 3 "~" H 7600 4600 50  0001 C CNN
 	1    7600 4600
@@
 P 7600 3950
 AR Path="/6194FDB3/61A37123" Ref="J?"  Part="1"
-AR Path="/6194FDB3/61A24149/61A37123" Ref="J27"  Part="1"
-F 0 "J27" H 7700 3650 50  0000 C CNN
+AR Path="/6194FDB3/61A24149/61A37123" Ref="J30"  Part="1"
+F 0 "J30" H 7700 3650 50  0000 C CNN
 F 1 "Conn_01x03_Male" H 7700 3750 50  0000 C CNN
-F 2 "" H 7600 3950 50  0001 C CNN
+F 2 "Connector_PinHeader_2.54mm:PinHeader_1x03_P2.54mm_Vertical" H 7600 3950 50  0001 C CNN
 F 3 "~" H 7600 3950 50  0001 C CNN
 	1    7600 3950
