File: SHIELD_MEGA/BAR.sch (KiCad schematic (older format))
At the start: 0 parts

Commit message: Barometer conections
Parts:
- added J73: Conn_01x06_Female, Connector_PinSocket_2.54mm:PinSocket_1x03_P2.54mm_Vertical, symbol Connector:Conn_01x06_Female
Connections:
- new net 3.3V: J73.6 (Pin_6)
- new net GND: J73.5 (Pin_5)
- new net SCL: J73.4 (Pin_4)
- new net SDA: J73.3 (Pin_3)
- no-connect marks 0 -> 2
Changed lines of the file:
@@
 Comment4 "LINCOLN WALLACE VELOSO ALMEIDA"
 $EndDescr
+$Comp
+L Connector:Conn_01x06_Female J73
+U 1 1 619D8F87
+P 5600 3600
+F 0 "J73" H 5492 3075 50  0000 C CNN
+F 1 "Conn_01x06_Female" H 5492 3166 50  0000 C CNN
+F 2 "Connector_PinSocket_2.54mm:PinSocket_1x03_P2.54mm_Vertical" H 5600 3600 50  0001 C CNN
+F 3 "~" H 5600 3600 50  0001 C CNN
+	1    5600 3600
+	-1   0    0    1
+$EndComp
+Wire Wire Line
+	6150 3300 5800 3300
+Text HLabel 6150 3300 2    50   Input ~ 0
+3.3V
+Text HLabel 6150 3400 2    50   Input ~ 0
+GND
+Wire Wire Line
+	6150 3400 5800 3400
+Wire Wire Line
+	5800 3500 6150 3500
+Text HLabel 6150 3500 2    50   Input ~ 0
+SCL
+Wire Wire Line
+	5800 3600 6150 3600
+Text HLabel 6150 3600 2    50   Input ~ 0
+SDA
+NoConn ~ 5800 3700
+NoConn ~ 5800 3800
 $EndSCHEMATC

Commit message: fixing footprint ref
Parts:
- J73: footprint Connector_PinSocket_2.54mm:PinSocket_1x03_P2.54mm_Vertical -> Connector_PinSocket_2.54mm:PinSocket_1x06_P2.54mm_Vertical
Changed lines of the file:
@@
 F 0 "J73" H 5492 3075 50  0000 C CNN
 F 1 "Conn_01x06_Female" H 5492 3166 50  0000 C CNN
-F 2 "Connector_PinSocket_2.54mm:PinSocket_1x03_P2.54mm_Vertical" H 5600 3600 50  0001 C CNN
+F 2 "Connector_PinSocket_2.54mm:PinSocket_1x06_P2.54mm_Vertical" H 5600 3600 50  0001 C CNN
 F 3 "~" H 5600 3600 50  0001 C CNN
 	1    5600 3600
